File: kicad/numitronbreakout.kicad_sch (KiCad schematic)
At the start: 12 parts, among them J1 Conn_01x06, U1 HV5812WG-G, U2 LM317_TO-220, U3 LM317_TO-220, U4 IV-12, U5 IV-12

Commit message: increased resistor size, generated gerbers for fab
Parts:
- C1: Manufacturer_Name (none) -> Samsung Electro-Mechanics; Manufacturer_Part_Number (none) -> CL31B104KBCNNNC
- PS1: MFR (none) -> MEAN WELL USA Inc.; Manufacturer_Name Mean Well -> MEAN WELL USA Inc.; Part No (none) -> LDB-600L
- R1, R3: footprint Resistor_SMD:R_0402_1005Metric_Pad0.72x0.64mm_HandSolder -> Resistor_SMD:R_1206_3216Metric_Pad1.30x1.75mm_HandSolder; Manufacturer_Name (none) -> Vishay Dale; Manufacturer_Part_Number (none) -> CRCW1206330RFKEA
- R2: footprint Resistor_SMD:R_0402_1005Metric_Pad0.72x0.64mm_HandSolder -> Resistor_SMD:R_1206_3216Metric_Pad1.30x1.75mm_HandSolder; Manufacturer_Name (none) -> Vishay Dale; Manufacturer_Part_Number (none) -> CRCW120668R0FKEA
- R4: footprint Resistor_SMD:R_0402_1005Metric_Pad0.72x0.64mm_HandSolder -> Resistor_SMD:R_1206_3216Metric_Pad1.30x1.75mm_HandSolder; Manufacturer_Name (none) -> Vishay Dale; Manufacturer_Part_Number (none) -> CRCW12061K00FKEA
- U1: Manufacturer_Name (none) -> Microchip Technology; Manufacturer_Part_Number (none) -> HV5812WG-G
- U2, U3: Manufacturer_Name (none) -> Texas Instruments; Manufacturer_Part_Number (none) -> LM317TNS/NOPB-ND
- U4, U5: now left out of the parts list
Changed lines of the file:
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@@
 			)
 		)
-		(property "Footprint" "Resistor_SMD:R_0402_1005Metric_Pad0.72x0.64mm_HandSolder"
+		(property "Footprint" "Resistor_SMD:R_1206_3216Metric_Pad1.30x1.75mm_HandSolder"
 			(at 161.036 49.784 90)
 			(effects
@@
 			)
 		)
-		(property "Description" "Resistor, US symbol"
+		(property "Description" "RES SMD 1K OHM 1% 1/4W 1206"
 			(at 160.02 49.53 0)
 			(effects
@@
 			)
 		)
+		(property "Manufacturer_Name" "Vishay Dale"
+			(at 160.02 49.53 0)
+			(effects
+				(font
+					(size 1.27 1.27)
+				)
+				(hide yes)
+			)
+		)
+		(property "Manufacturer_Part_Number" "CRCW12061K00FKEA"
+			(at 160.02 49.53 0)
+			(effects
+				(font
+					(size 1.27 1.27)
+				)
+				(hide yes)
+			)
+		)
 		(pin "2"
 		)
@@
 			)
 		)
-		(property "Description" "1.5A 35V Adjustable Linear Regulator, TO-220"
+		(property "Description" "IC REG LIN POS ADJ 1.5A TO220-3"
 			(at 88.9 38.1 0)
 			(effects
@@
 			)
 		)
+		(property "Manufacturer_Name" "Texas Instruments"
+			(at 88.9 38.1 0)
+			(effects
+				(font
+					(size 1.27 1.27)
+				)
+				(hide yes)
+			)
+		)
+		(property "Manufacturer_Part_Number" "LM317TNS/NOPB-ND"
+			(at 88.9 38.1 0)
+			(effects
+				(font
+					(size 1.27 1.27)
+				)
+				(hide yes)
+			)
+		)
 		(pin "3"
 		)
@@
 		)
 		(property "Part No" "HV5812WG-G"
+			(at 63.5 109.22 0)
+			(effects
+				(font
+					(size 1.27 1.27)
+				)
+				(hide yes)
+			)
+		)
+		(property "Manufacturer_Name" "Microchip Technology"
+			(at 63.5 109.22 0)
+			(effects
+				(font
+					(size 1.27 1.27)
+				)
+				(hide yes)
+			)
+		)
+		(property "Manufacturer_Part_Number" "HV5812WG-G"
 			(at 63.5 109.22 0)
 			(effects
@@
 			)
 		)
-		(property "Footprint" "Resistor_SMD:R_0402_1005Metric_Pad0.72x0.64mm_HandSolder"
+		(property "Footprint" "Resistor_SMD:R_1206_3216Metric_Pad1.30x1.75mm_HandSolder"
 			(at 97.536 49.784 90)
 			(effects
@@
 			)
 		)
-		(property "Description" "Resistor, US symbol"
+		(property "Description" "RES SMD 68 OHM 1% 1/4W 1206"
 			(at 96.52 49.53 0)
 			(effects
@@
 		)
 		(property "Part No" "CRCW040248R7FKED"
+			(at 96.52 49.53 0)
+			(effects
+				(font
+					(size 1.27 1.27)
+				)
+				(hide yes)
+			)
+		)
+		(property "Manufacturer_Name" "Vishay Dale"
+			(at 96.52 49.53 0)
+			(effects
+				(font
+					(size 1.27 1.27)
+				)
+				(hide yes)
+			)
+		)
+		(property "Manufacturer_Part_Number" "CRCW120668R0FKEA"
 			(at 96.52 49.53 0)
 			(effects
@@
 			)
 		)
-		(property "Footprint" "Resistor_SMD:R_0402_1005Metric_Pad0.72x0.64mm_HandSolder"
+		(property "Footprint" "Resistor_SMD:R_1206_3216Metric_Pad1.30x1.75mm_HandSolder"
 			(at 97.536 42.164 90)
 			(effects
@@
 			)
 		)
-		(property "Description" "Resistor, US symbol"
+		(property "Description" "RES SMD 330 OHM 1% 1/4W 1206"
 			(at 96.52 41.91 0)
 			(effects
@@
 			)
 		)
+		(property "Manufacturer_Name" "Vishay Dale"
+			(at 96.52 41.91 0)
+			(effects
+				(font
+					(size 1.27 1.27)
+				)
+				(hide yes)
+			)
+		)
+		(property "Manufacturer_Part_Number" "CRCW1206330RFKEA"
+			(at 96.52 41.91 0)
+			(effects
+				(font
+					(size 1.27 1.27)
+				)
+				(hide yes)
+			)
+		)
 		(pin "2"
 		)
@@
 			)
 		)
-		(property "Datasheet" "~"
+		(property "Datasheet" "https://mm.digikey.com/Volume0/opasdata/d220001/medias/docus/1256/CL31B104KBCNNNC_Spec.pdf"
 			(at 130.81 91.44 0)
 			(effects
@@
 			)
 		)
-		(property "Description" "Unpolarized capacitor"
+		(property "Description" "CAP CER 0.1UF 50V X7R 1206"
 			(at 130.81 91.44 0)
 			(effects
@@
 		)
 		(property "Part No" ""
+			(at 130.81 91.44 0)
+			(effects
+				(font
+					(size 1.27 1.27)
+				)
+				(hide yes)
+			)
+		)
+		(property "Manufacturer_Name" "Samsung Electro-Mechanics"
+			(at 130.81 91.44 0)
+			(effects
+				(font
+					(size 1.27 1.27)
+				)
+				(hide yes)
+			)
+		)
+		(property "Manufacturer_Part_Number" "CL31B104KBCNNNC"
 			(at 130.81 91.44 0)
 			(effects
@@
 		(unit 1)
 		(exclude_from_sim no)
-		(in_bom yes)
+		(in_bom no)
 		(on_board yes)
 		(dnp no)
@@
 			)
 		)
-		(property "Description" "1.5A 35V Adjustable Linear Regulator, TO-220"
+		(property "Description" "IC REG LIN POS ADJ 1.5A TO220-3"
 			(at 152.4 38.1 0)
 			(effects
@@
 		)
 		(property "Part No" "LM317TNS/NOPB-ND"
+			(at 152.4 38.1 0)
+			(effects
+				(font
+					(size 1.27 1.27)
+				)
+				(hide yes)
+			)
+		)
+		(property "Manufacturer_Name" "Texas Instruments"
+			(at 152.4 38.1 0)
+			(effects
+				(font
+					(size 1.27 1.27)
+				)
+				(hide yes)
+			)
+		)
+		(property "Manufacturer_Part_Number" "LM317TNS/NOPB-ND"
 			(at 152.4 38.1 0)
 			(effects
@@
 			)
 		)
-		(property "Footprint" "Resistor_SMD:R_0402_1005Metric_Pad0.72x0.64mm_HandSolder"
+		(property "Footprint" "Resistor_SMD:R_1206_3216Metric_Pad1.30x1.75mm_HandSolder"
 			(at 161.036 42.164 90)
 			(effects
@@
 			)
 		)
-		(property "Description" "Resistor, US symbol"
+		(property "Description" "RES SMD 330 OHM 1% 1/4W 1206"
 			(at 160.02 41.91 0)
 			(effects
@@
 		)
 		(property "Part No" "CRCW0402240RFKED"
+			(at 160.02 41.91 0)
+			(effects
+				(font
+					(size 1.27 1.27)
+				)
+				(hide yes)
+			)
+		)
+		(property "Manufacturer_Name" "Vishay Dale"
+			(at 160.02 41.91 0)
+			(effects
+				(font
+					(size 1.27 1.27)
+				)
+				(hide yes)
+			)
+		)
+		(property "Manufacturer_Part_Number" "CRCW1206330RFKEA"
 			(at 160.02 41.91 0)
 			(effects
@@
 		(unit 1)
 		(exclude_from_sim no)
-		(in_bom yes)
+		(in_bom no)
 		(on_board yes)
 		(dnp no)
@@
 			)
 		)
-		(property "Description" "LED Power Supplies 9-28Vin 2-30Vout 600mA pin style"
+		(property "Description" "LED DVR CC BUCK-BST 2-30V 600MA"
 			(at 191.77 38.1 0)
 			(effects
@@
 			)
 		)
-		(property "Manufacturer_Name" "Mean Well"
+		(property "Manufacturer_Name" "MEAN WELL USA Inc."
 			(at 223.52 50.8 0)
 			(effects
@@
 				(hide yes)
 			)
+		)
+		(property "MFR" "MEAN WELL USA Inc."
+			(at 191.77 38.1 0)
+			(effects
+				(font
+					(size 1.27 1.27)
+				)
+				(hide yes)
+			)
+		)
+		(property "Part No" "LDB-600L"
+			(at 191.77 38.1 0)
+			(effects
+				(font
+					(size 1.27 1.27)
+				)
+				(hide yes)
+			)
