File: kicad/numitronbreakout.kicad_pcb (KiCad board)
At the start: 4 copper layers, 60 x 100 mm, 17 parts, among them J1 Conn_01x06, U1 HV5812WG-G, U2 LM317_TO-220, U3 LM317_TO-220, U4 IV-12, U5 IV-12

Commit message: Small routing fix
Parts:
- M3 SCREW: renamed from REF**
- moved R5 0.05 mm to (136.6, 90.0)
Changed lines of the file:
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@@
 			(at 0 -4.2 0)
 			(layer "F.SilkS")
+			(hide yes)
 			(effects
 				(font
@@
 	(footprint "Resistor_SMD:R_1206_3216Metric_Pad1.30x1.75mm_HandSolder"
 		(layer "F.Cu")
-		(at 136.5 90)
+		(at 136.55 90)
 		(descr "Resistor SMD 1206 (3216 Metric), square (rectangular) end terminal, IPC_7351 nominal with elongated pad for handsoldering. (Body size source: IPC-SM-782 page 72, https://www.pcb-3d.com/wordpress/wp-content/uploads/ipc-sm-782a_amendment_1_and_2.pdf), generated with kicad-footprint-generator")
 		(tags "resistor handsolder")
@@
 		(descr "Mounting Hole 3.2mm, M3")
 		(tags "mounting hole 3.2mm m3")
-		(property "Reference" "REF**"
+		(property "Reference" "M3 SCREW"
 			(at 0 -4.2 0)
 			(layer "F.SilkS")
@@
 			(at 0 -4.2 0)
 			(layer "F.SilkS")
+			(hide yes)
 			(effects
 				(font
@@
 			(at 0 -4.2 0)
 			(layer "F.SilkS")
+			(hide yes)
 			(effects
 				(font
@@
 	)
 	(segment
-		(start 146.42 103.08)
-		(end 146.42 63)
+		(start 142.5 108)
+		(end 142.5 105.5)
 		(width 0.6)
 		(layer "B.Cu")
@@
 	)
 	(segment
-		(start 142.5 107)
-		(end 146.42 103.08)
+		(start 146.42 101.58)
+		(end 146.42 63)
 		(width 0.6)
 		(layer "B.Cu")
@@
 	)
 	(segment
-		(start 142.5 108)
-		(end 142.5 107)
+		(start 142.5 105.5)
+		(end 146.42 101.58)
 		(width 0.6)
 		(layer "B.Cu")
@@
 	)
 	(segment
-		(start 132.44 87.94)
-		(end 134.5 90)
+		(start 132.44 83.12)
+		(end 132.44 77.06)
 		(width 0.6)
 		(layer "F.Cu")
@@
 	)
 	(segment
-		(start 132.44 83.12)
-		(end 132.44 77.06)
+		(start 132.44 87.94)
+		(end 134.5 90)
 		(width 0.6)
 		(layer "F.Cu")
@@
 	)
 	(segment
-		(start 149 70)
-		(end 154.04 64.96)
+		(start 134.5 90)
+		(end 135 90)
 		(width 0.6)
 		(layer "F.Cu")
@@
 	)
 	(segment
-		(start 134.5 90)
-		(end 134.95 90)
+		(start 149 70)
+		(end 154.04 64.96)
 		(width 0.6)
 		(layer "F.Cu")
@@
 	)
 	(segment
-		(start 140 90)
-		(end 138.55 90)
+		(start 138.1 90)
+		(end 140 90)
 		(width 0.6)
 		(layer "F.Cu")
