File: controller/numitroncontrol.kicad_pcb (KiCad board)
At the start: 4 copper layers, 35 x 100 mm, 9 parts, among them J0 Screw_Terminal_01x02, J1 Conn_01x06, J2 Conn_01x06, J3 RTC, J4 GPS, U1 LM317_TO-220

Commit message: control pcb finished
Parts:
- added ?: , , F.Cu at (106.5, 124.6)
- added ?: , , F.Cu at (106.5, 111.9)
- added ?: , , F.Cu at (106.5, 109.3)
- added ?: , , F.Cu at (129.4, 86.8)
- added ?: , , F.Cu at (106.5, 106.8)
- added ?: , , F.Cu at (106.5, 84.3)
- added ?: , , F.Cu at (129.4, 91.9)
- added ?: , , F.Cu at (106.5, 119.5)
- added ?: , , F.Cu at (106.5, 117.0)
- added ?: , , F.Cu at (129.4, 81.8)
- added ?: , , F.Cu at (129.4, 84.3)
- added ?: , , F.Cu at (106.5, 122.0)
- added ?: , , F.Cu at (106.5, 114.4)
- added ?: , , F.Cu at (129.4, 89.4)
- added J3: PTH, Qwiic GPS - Titan X1 v10:1X04_NO_SILK, F.Cu at (106.5, 84.3)
- added J5: , Qwiic GPS - Titan X1 v10:1X01_NO_SILK, F.Cu at (106.5, 81.8)
- added REF**: MountingHole_3.2mm_M3_Pad, MountingHole:MountingHole_3.2mm_M3_Pad, F.Cu at (150.0, 53.5)
- added REF**: MountingHole_3.2mm_M3_Pad, MountingHole:MountingHole_3.2mm_M3_Pad, F.Cu at (150.0, 146.5)
- moved J4 20.0 mm to (135.0, 105.0)
- moved J3 12.5 mm to (135.0, 82.5)
- moved A1 9.00 mm to (150.1, 75.2)
- moved U1 8.87 mm to (154.9, 63.5)
- moved R1 8.87 mm to (155.0, 69.5)
- moved R2 8.87 mm to (160.0, 69.5)
- moved J0 4.83 mm to (138.2, 60.0)
- moved J2 4.77 mm to (150.0, 136.5)
- moved J1 0.77 mm to (150.0, 125.5)
Routing:
- net BLANKING: track 91.9 -> 71.2 mm
- net STROBE: track 58.3 -> 76.5 mm, vias 1 -> 2
- net CLOCK: track 51.0 -> 68.8 mm, vias 1 -> 2
- net DIMMING: track 58.9 -> 76.4 mm, vias 1 -> 2
- net D_IN: track 52.7 -> 37.4 mm
- net +3V3: track 25.4 -> 38.3 mm
- net +12V: track 117.4 -> 104.9 mm, vias 0 -> 1
- net SCL: track 23.0 -> 29.7 mm, vias 1 -> 0
- net SDA: track 23.1 -> 29.0 mm, vias 1 -> 0
- net Net-(J1-Pin_2): track 19.8 -> 14.9 mm
- net Net-(J0-Pin_1): track 27.5 -> 25.7 mm
Other:
- board text added: "IV-12 NUMITRON CONTROL BOARD A. LEVINE REV.01"
- board text added: "JLCJLCJLCJLC"

Commit message: control pcb edits
Parts:
- moved J4 5.00 mm to (135.0, 110.0)
- moved ? 3.20 mm to (106.5, 127.8)
- moved ? 3.20 mm to (106.5, 115.1)
- moved ? 3.20 mm to (106.5, 112.5)
- moved ? 3.20 mm to (106.5, 110.0)
- moved ? 3.20 mm to (106.5, 122.7)
- moved ? 3.20 mm to (106.5, 120.2)
- moved ? 3.20 mm to (106.5, 117.6)
- moved ? 3.20 mm to (106.5, 125.2)
Routing:
- net SDA: track 29.0 -> 33.7 mm
- net +3V3: track 38.3 -> 43.1 mm
- net SCL: track 29.7 -> 34.2 mm
- net Net-(J0-Pin_1): track 25.7 -> 24.9 mm
