File: controller/numitroncontrol.kicad_pcb (KiCad board)
At the start: 4 copper layers, 35 x 100 mm, 27 parts, among them J0 Screw_Terminal_01x02, J1 Conn_01x06, J2 Conn_01x06, J3 PTH, J3 RTC, J4 GPS, U1 LM317_TO-220

Commit message: played tetris on pcb and re-exported prod files
Parts:
- added RV1: R_Potentiometer_US, Connector_PinHeader_2.54mm:PinHeader_1x03_P2.54mm_Vertical, F.Cu at (137.4, 70.0)
- moved J0 3.40 mm to (138.2, 63.4)
- moved R1 2.95 mm to (157.5, 68.0)
- moved R2 2.95 mm to (162.5, 68.0)
- moved U1 2.54 mm to (157.5, 63.5)
Routing:
- net +5V: track 0.00 -> 39.9 mm
- net POT: track 0.00 -> 37.1 mm
- net D_IN: track 37.4 -> 34.5 mm
- net Net-(U1-ADJ): track 10.0 -> 8.52 mm
- net Net-(J0-Pin_1): track 24.9 -> 26.3 mm
- net +12V: track 104.9 -> 104.3 mm
- net GND: track 1.92 -> 2.42 mm
