File: controller/numitroncontrol.kicad_pcb (KiCad board)
At the start: 4 copper layers, 35 x 100 mm, 12 parts, among them J0 Screw_Terminal_01x02, J1 Conn_01x06, J2 Conn_01x06, J3 RTC, J4 Screw_Terminal_01x03, J5 Conn_01x03_Pin, U1 LM317_TO-220

Commit message: more controller layout updates
Parts:
- J0: footprint TerminalBlock_4Ucon:TerminalBlock_4Ucon_1x02_P3.50mm_Horizontal -> TerminalBlock_TE-Connectivity:TerminalBlock_TE_282834-2_1x02_P2.54mm_Horizontal
- J3: value RTC -> I2C
- moved J0 3.81 mm to (114.3, 92.7), turned to -90 degrees
- moved R1 1.38 mm to (133.4, 99.8)
- moved R2 1.38 mm to (138.4, 99.8)
- moved U1 1.38 mm to (133.3, 95.2)
Connections:
- REF** pad 1: (no net) -> GND (x2)
Routing:
- net Net-(J0-Pin_1): track 27.3 -> 25.2 mm
- net DIMMING: track 76.3 -> 78.3 mm
- net D_IN2: track 35.2 -> 36.8 mm
- net STROBE: track 76.7 -> 78.1 mm
- net +12V: track 109.1 -> 107.9 mm
- net BLANKING: track 73.7 -> 74.3 mm
- net CLOCK: track 71.6 -> 72.2 mm
Other:
- board text added: "CONTROL"
- board text added: "DIMMER"
- board text added: "I2C"

Commit message: layout updates, gerbers generated
Parts:
- J5: footprint Connector_PinSocket_2.54mm:PinSocket_1x03_P2.54mm_Vertical -> Connector_PinHeader_2.54mm:PinHeader_1x03_P2.54mm_Vertical
Other:
- board text added: "BREAKOUT 1"
- board text added: "BREAKOUT 2"
- board text added: "VIN"
Changed lines of the file:
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@@
 			(outputformat 1)
 			(mirror no)
-			(drillshape 1)
+			(drillshape 0)
 			(scaleselection 1)
-			(outputdirectory "")
+			(outputdirectory "production/")
 		)
 	)
@@
 			(at -5.22 3.81 0)
 			(layer "F.Fab")
+			(hide yes)
 			(effects
 				(font
@@
 		(tags "TO-220-3 Vertical RM 2.54mm")
 		(property "Reference" "U1"
-			(at 2.54 -4.27 0)
+			(at -1.905 -4.27 0)
 			(layer "F.SilkS")
 			(effects
@@
 		)
 		(property "Value" "LM317_TO-220"
-			(at 2.54 2.5 0)
+			(at 2.54 -2.54 0)
 			(layer "F.Fab")
 			(effects
@@
 		)
 		(fp_text user "${REFERENCE}"
-			(at 2.54 -4.27 0)
+			(at -1.905 -4.27 0)
 			(layer "F.Fab")
 			(effects
@@
 		(tags "Through hole pin header THT 1x04 2.54mm single row")
 		(property "Reference" "J3"
-			(at 0 -2.33 0)
+			(at 0 -2.54 0)
 			(layer "F.SilkS")
 			(effects
@@
 		)
 		(property "Value" "I2C"
-			(at 0 9.95 0)
+			(at 2.54 3.81 90)
 			(layer "F.Fab")
+			(hide yes)
 			(effects
 				(font
@@
 		)
 		(fp_text user "${REFERENCE}"
-			(at 0 3.81 90)
+			(at 0 -2.54 180)
 			(layer "F.Fab")
 			(effects
@@
 		)
 		(property "Value" "MountingHole_3.2mm_M3_Pad"
-			(at 0 10.55 0)
+			(at 0.12 4.618 0)
 			(layer "F.Fab")
 			(effects
@@
 		(tags "THT Terminal Block TE 282834-2 pitch 2.54mm size 5.54x6.5mm drill 1.1mm pad 2.1mm")
 		(property "Reference" "J0"
-			(at 5.08 -2.54 0)
+			(at -2.54 2.54 0)
 			(layer "F.SilkS")
 			(effects
@@
 		)
 		(property "Value" "Screw_Terminal_01x02"
-			(at 1.27 4.37 90)
+			(at 5.08 0 180)
 			(layer "F.Fab")
+			(hide yes)
 			(effects
 				(font
@@
 		)
 		(fp_text user "${REFERENCE}"
-			(at 1.27 2 90)
+			(at -2.54 2.54 180)
 			(layer "F.Fab")
 			(effects
@@
 		(property "Value" "Arduino_Nano_RP2040_Connect_Socket"
 			(at 0 -21.082 90)
-			(layer "F.Fab")
+			(layer "F.SilkS")
 			(effects
 				(font
@@
 		(tags "resistor handsolder")
 		(property "Reference" "R2"
-			(at 0 -1.65 90)
+			(at 0 1.865 90)
 			(layer "F.SilkS")
 			(effects
@@
 		)
 		(property "Value" "3.3 kΩ"
-			(at 0 1.65 90)
+			(at 2.485 -0.675 180)
 			(layer "F.Fab")
 			(effects
@@
 		)
 		(property "Value" "390 Ω"
-			(at 0 1.65 90)
+			(at -2.485 -0.675 180)
 			(layer "F.Fab")
 			(effects
@@
 		(embedded_fonts no)
 	)
-	(footprint "Connector_PinSocket_2.54mm:PinSocket_1x03_P2.54mm_Vertical"
+	(footprint "Connector_PinHeader_2.54mm:PinHeader_1x03_P2.54mm_Vertical"
 		(layer "F.Cu")
 		(at 114.3 158.115 180)
-		(descr "Through hole straight socket strip, 1x03, 2.54mm pitch, single row (from Kicad 4.0.7), script generated")
-		(tags "Through hole socket strip THT 1x03 2.54mm single row")
+		(descr "Through hole straight pin header, 1x03, 2.54mm pitch, single row")
+		(tags "Through hole pin header THT 1x03 2.54mm single row")
 		(property "Reference" "J5"
-			(at 0 7.62 0)
+			(at 0 7.62 180)
 			(layer "F.SilkS")
 			(effects
@@
 		)
 		(property "Value" "Conn_01x03_Pin"
-			(at 0 7.85 0)
+			(at -2.54 2.54 270)
 			(layer "F.Fab")
+			(hide yes)
 			(effects
 				(font
@@
 		)
 		(fp_line
-			(start 1.33 -1.33)
-			(end 1.33 0)
+			(start -1.33 6.41)
+			(end 1.33 6.41)
 			(stroke
 				(width 0.12)
@@
 		)
 		(fp_line
-			(start 0 -1.33)
-			(end 1.33 -1.33)
+			(start -1.33 1.27)
+			(end 1.33 1.27)
 			(stroke
 				(width 0.12)
@@
 		)
 		(fp_line
-			(start -1.33 6.41)
-			(end 1.33 6.41)
+			(start -1.33 1.27)
+			(end -1.33 6.41)
 			(stroke
 				(width 0.12)
@@
 		)
 		(fp_line
-			(start -1.33 1.27)
-			(end 1.33 1.27)
+			(start -1.33 0)
+			(end -1.33 -1.33)
 			(stroke
 				(width 0.12)
@@
 		)
 		(fp_line
-			(start -1.33 1.27)
-			(end -1.33 6.41)
+			(start -1.33 -1.33)
+			(end 0 -1.33)
 			(stroke
 				(width 0.12)
@@
 		)
 		(fp_line
-			(start 1.75 6.85)
-			(end -1.8 6.85)
+			(start 1.8 6.85)
+			(end 1.8 -1.8)
 			(stroke
 				(width 0.05)
@@
 		)
 		(fp_line
-			(start 1.75 -1.8)
-			(end 1.75 6.85)
+			(start 1.8 -1.8)
+			(end -1.8 -1.8)
 			(stroke
 				(width 0.05)
@@
 		(fp_line
 			(start -1.8 6.85)
-			(end -1.8 -1.8)
+			(end 1.8 6.85)
 			(stroke
 				(width 0.05)
@@
 		(fp_line
 			(start -1.8 -1.8)
-			(end 1.75 -1.8)
+			(end -1.8 6.85)
 			(stroke
 				(width 0.05)
@@
 		)
 		(fp_line
-			(start 1.27 -0.635)
+			(start 1.27 -1.27)
 			(end 1.27 6.35)
 			(stroke
@@
 		)
 		(fp_line
-			(start 0.635 -1.27)
-			(end 1.27 -0.635)
+			(start -0.635 -1.27)
+			(end 1.27 -1.27)
 			(stroke
 				(width 0.1)
@@
 		(fp_line
 			(start -1.27 6.35)
-			(end -1.27 -1.27)
+			(end -1.27 -0.635)
 			(stroke
 				(width 0.1)
@@
 		)
 		(fp_line
-			(start -1.27 -1.27)
-			(end 0.635 -1.27)
+			(start -1.27 -0.635)
+			(end -0.635 -1.27)
 			(stroke
 				(width 0.1)
@@
 		)
 		(fp_text user "${REFERENCE}"
-			(at 0 2.54 90)
+			(at 0 7.62 0)
 			(layer "F.Fab")
 			(effects
@@
 		)
 		(embedded_fonts no)
-		(model "${KICAD9_3DMODEL_DIR}/Connector_PinSocket_2.54mm.3dshapes/PinSocket_1x03_P2.54mm_Vertical.wrl"
+		(model "${KICAD9_3DMODEL_DIR}/Connector_PinHeader_2.54mm.3dshapes/PinHeader_1x03_P2.54mm_Vertical.wrl"
 			(offset
 				(xyz 0 0 0)
@@
 		)
 		(property "Value" "Screw_Terminal_01x03"
-			(at 0 7.41 0)
+			(at -2.54 2.54 270)
 			(layer "F.Fab")
+			(hide yes)
 			(effects
 				(font
@@
 		)
 		(fp_text user "${REFERENCE}"
-			(at 0 2.54 90)
+			(at 0 7.62 180)
 			(layer "F.Fab")
 			(effects
@@
 			(at -5.22 3.835 0)
 			(layer "F.Fab")
+			(hide yes)
 			(effects
 				(font
@@
 		)
 	)
+	(gr_text "BREAKOUT 1"
+		(at 135.89 150.495 0)
+		(layer "F.SilkS")
+		(effects
+			(font
+				(size 1 1)
+				(thickness 0.2)
+				(bold yes)
+			)
+			(justify right)
+		)
+	)
 	(gr_text "CONTROL"
 		(at 111.76 151.13 270)
@@
 		)
 	)
+	(gr_text "VIN"
+		(at 118.11 90.17 0)
+		(layer "F.SilkS")
+		(effects
+			(font
+				(size 1 1)
+				(thickness 0.2)
+				(bold yes)
+			)
+			(justify right)
+		)
+	)
 	(gr_text "I2C"
 		(at 111.76 120.65 270)
@@
 		)
 	)
+	(gr_text "BREAKOUT 2"
+		(at 135.89 161.925 0)
+		(layer "F.SilkS")
+		(effects
+			(font
+				(size 1 1)
+				(thickness 0.2)
+				(bold yes)
+			)
+			(justify right)
+		)
+	)
 	(gr_text_box "1 D_IN		2 D_OUT\n3 BLANKING	4 CLOCK\n5 STROBE	6 DIMMING\n7 12V		8 GND"
 		(start 111.55 172.45)
@@
 		)
 	)
-	(gr_text_box "+		-"
+	(gr_text_box "- 12V +"
 		(start 118.63 91.31125)
 		(end 120.13 96.64875)
@@
 				(thickness 0.1)
 			)
-			(justify top mirror)
+			(justify top)
 		)
 		(border yes)
@@
 	(segment
 		(start 138.39 100.75)
-		(end 136.39 100.75)
+		(end 136.74 100.75)
+		(width 0.75)
+		(layer "F.Cu")
+		(net 7)
+	)
+	(segment
+		(start 136.74 100.75)
+		(end 136.525 100.965)
 		(width 0.75)
 		(layer "F.Cu")
@@
 	)
 	(via
-		(at 136.39 100.75)
-		(size 0.6)
-		(drill 0.3)
+		(at 136.525 100.965)
+		(size 1)
+		(drill 0.75)
 		(layers "F.Cu" "B.Cu")
 		(net 7)
